Commit message: Added the Wheels

File: robot.urdf (robot description, URDF)
Before this commit: robot SBR, 1 links, 0 joints
Links:
- added link left_wheel; visual mesh filename=file:///home/drak/ros2_ws/src/cadtoURDF/meshes/left_wheel.S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
- added link right_wheel; visual mesh filename=file:///home/drak/ros2_ws/src/cadtoURDF/meshes/right_wheel.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
Joints:
- added joint base_left_wheel_joint: type continuous, parent base_link, child left_wheel, origin xyz=0 0 0 rpy=0 0 0, axis 0 1 0
- added joint base_right_wheel_joint: type continuous, parent base_link, child right_wheel, origin xyz=0 0 0 rpy=0 0 0, axis 0 1 0

Commit message: Added a base_footprint and a world

File: robot.urdf (robot description, URDF)
Before this commit: robot SBR, 3 links, 2 joints
Links:
- added link base_footprint
- added link world_link; visual mesh filename=file:///home/drak/ros2_ws/src/cadtoURDF/meshes/world.STL
Joints:
- added joint base_footprint_world_joint: type fixed, parent base_footprint, child world_link, origin xyz=0 0 -1.7 rpy=0 0 0
- added joint base_joint: type fixed, parent base_link, child base_footprint, origin xyz=0 0 -0.350 rpy=0 0 0
